File: Урок 7/ДЗ 7/ДЗ 7.kicad_sch (KiCad schematic)
At the start: 22 parts, among them SW1 SW_Push, SW2 SW_Push

Commit message: 1
Parts:
- added Q3: ~, cadstarpcblib:BC32725PBFREE, symbol My_lib2:BC327-25_PBFREE
- added R2: 10k, symbol Device:R
- added U1: ~, symbol My_lib2:PC817X3NSZ9F
- renumbered R7 to R1
Connections:
- net GND: now also U1.2 (Cathode), U1.3 (Emitter); no longer D1.2 (A), Q1.3 (A)
- net at R1.2: now also U1.1 (Anode)
- new net: Q3.2 (B), R2.2
- new net +5V: R2.1, U1.4 (Collector)

Commit message: 1
Parts:
- removed BZ1: Buzzer, symbol Device:Buzzer
- removed D1: 5.1V, Diode_THT:D_DO-41_SOD81_P10.16mm_Horizontal, symbol Diode:1N47xxA
- removed D3, D4, D5, D6: IR204A, LED_THT:LED_D3.0mm_IRBlack, symbol LED:IR204A
- removed Q1, Q2: ~, cadstarpcblib:BC32725PBFREE, symbol My_lib2:BC327-25_PBFREE
- removed R1, R2: 10k, symbol Device:R
- removed R1, R2, R6: 3k, symbol Device:R
- removed R2: 1k, symbol Device:R
- removed R3: 4k, symbol Device:R_Potentiometer
- removed SW1: SW_Push, symbol Switch:SW_Push
- added D1: 1N4007, Diode_THT:D_DO-41_SOD81_P10.16mm_Horizontal, symbol Diode:1N4007
- added K1: HONGFA_HFD2-0xx-x-L2-x, Relay_THT:Relay_DPDT_Omron_G6AK, symbol Relay:HONGFA_HFD2-0xx-x-L2-x
- added R2: 10k, symbol Device:R
- LA1: value 250mA -> Lamp
- R3, R4, R5: value 3k -> 10k
- renumbered Q3 to Q1
Connections:
- net +12V: now also K1.11, K1.21; no longer LA1.2 (+)
- net +5V: now also R5.2; no longer U1.4 (Collector)
- net 5V: now also Q1.3 (A)
- net GND: now also LA1.2 (+), R4.2; no longer D2.1 (K)
- net at D2.2 (A): now also Q1.1 (C), D1.1 (K), K1.B1
- net at LA1.1 (-): now also K1.14
- net at Q1.2 (B): now also R2.1
- net at R3.2: now also R4.1, D1.2 (A), K1.A1
- new net: R2.2, R5.1, U1.4 (Collector)
- new net: D2.1 (K), R3.1
Other:
- moved on the sheet: Q1, R1, SW2, U1

Commit message: 1
Parts:
- removed R4: 10k, symbol Device:R
Connections:
- net GND: now also D1.2 (A), K1.A1, R3.2
Changed lines of the file:
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@@
+	)
+	(junction
+		(at 104.14 63.5)
+		(diameter 0)
+		(color 0 0 0 0)
 	)
 	(junction
@@
 	)
 	(junction
-		(at 104.14 63.5)
-		(diameter 0)
-		(color 0 0 0 0)
-	)
-	(junction
 		(at 87.63 83.82)
 		(diameter 0)
@@
 	(wire
 		(pts
-			(xy 104.14 44.45) (xy 104.14 48.26)
+			(xy 104.14 44.45) (xy 104.14 63.5)
 		)
 		(stroke
@@
 		(pts
 			(xy 104.14 63.5) (xy 104.14 66.04)
-		)
-		(stroke
-			(width 0)
-			(type default)
-		)
-	)
-	(wire
-		(pts
-			(xy 104.14 55.88) (xy 104.14 63.5)
 		)
 		(stroke
@@
 					(unit 1)
 				)
-			)
-		)
-	)
-	(symbol
-		(lib_id "Device:R")
-		(at 104.14 52.07 180)
-		(unit 1)
-		(exclude_from_sim no)
-		(in_bom yes)
-		(on_board yes)
-		(dnp no)
-		(fields_autoplaced yes)
-		(property "Reference" "R4"
-			(at 106.68 50.7999 0)
-			(effects
-				(font
-					(size 1.27 1.27)
-				)
-				(justify right)
-			)
-		)
-		(property "Value" "10k"
-			(at 106.68 53.3399 0)
-			(effects
-				(font
-					(size 1.27 1.27)
-				)
-				(justify right)
-			)
-		)
-		(property "Footprint" ""
-			(at 105.918 52.07 90)
-			(effects
-				(font
-					(size 1.27 1.27)
-				)
-				(hide yes)
-			)
-		)
-		(property "Datasheet" "~"
-			(at 104.14 52.07 0)
-			(effects
-				(font
-					(size 1.27 1.27)
-				)
-				(hide yes)
-			)
-		)
-		(property "Description" "Resistor"
-			(at 104.14 52.07 0)
-			(effects
-				(font
-					(size 1.27 1.27)
-				)
-				(hide yes)
-			)
-		)
-		(pin "1"
-		)
-		(pin "2"
-		)
-		(instances
-			(project "ДЗ 7"
-				(path "/c8a16ae6-9a59-46d9-90dc-31792699b8d1"
-					(reference "R4")
-					(unit 1)
-				)

Commit message: 1
Parts:
- R1, R5: value 10k -> 180
- R3: value 10k -> 500
Changed lines of the file:
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@@
 			)
 		)
-		(property "Value" "10k"
+		(property "Value" "500"
 			(at 78.74 69.8499 0)
 			(effects
@@
 			)
 		)
-		(property "Value" "10k"
+		(property "Value" "180"
 			(at 53.34 96.52 90)
 			(effects
@@
 			)
 		)
-		(property "Value" "10k"
+		(property "Value" "180"
 			(at 72.39 101.5999 0)
 			(effects

Commit message: 1
Parts:
- R1: value 180 -> 100
- R3: value 500 -> 150
Changed lines of the file:
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@@
 	)
 	(junction
-		(at 63.5 130.81)
+		(at 63.5 146.05)
 		(diameter 0)
 		(color 0 0 0 0)
@@
 	(wire
 		(pts
-			(xy 57.15 130.81) (xy 63.5 130.81)
+			(xy 57.15 146.05) (xy 63.5 146.05)
 		)
 		(stroke
@@
 	(wire
 		(pts
-			(xy 57.15 100.33) (xy 57.15 113.03)
+			(xy 57.15 100.33) (xy 57.15 128.27)
 		)
 		(stroke
@@
 	(wire
 		(pts
-			(xy 69.85 109.22) (xy 69.85 113.03)
+			(xy 69.85 109.22) (xy 69.85 128.27)
 		)
 		(stroke
@@
 	(wire
 		(pts
-			(xy 63.5 130.81) (xy 69.85 130.81)
+			(xy 63.5 146.05) (xy 69.85 146.05)
 		)
 		(stroke
@@
 	(wire
 		(pts
-			(xy 57.15 130.81) (xy 57.15 125.73)
+			(xy 57.15 146.05) (xy 57.15 140.97)
 		)
 		(stroke
@@
 	(wire
 		(pts
-			(xy 69.85 130.81) (xy 69.85 125.73)
+			(xy 69.85 146.05) (xy 69.85 140.97)
 		)
 		(stroke
@@
 	(symbol
 		(lib_id "My_lib2:PC817X3NSZ9F")
-		(at 67.31 119.38 0)
+		(at 67.31 134.62 0)
 		(unit 1)
 		(exclude_from_sim no)
@@
 		(fields_autoplaced yes)
 		(property "Reference" "U1"
-			(at 73.66 118.7449 0)
+			(at 73.66 133.9849 0)
 			(effects
 				(font
@@
 		)
 		(property "Value" "~"
-			(at 73.66 120.65 0)
+			(at 73.66 135.89 0)
 			(effects
 				(font
@@
 		)
 		(property "Footprint" ""
-			(at 67.31 119.38 0)
+			(at 67.31 134.62 0)
 			(effects
 				(font
@@
 		)
 		(property "Datasheet" ""
-			(at 67.31 119.38 0)
+			(at 67.31 134.62 0)
 			(effects
 				(font
@@
 		)
 		(property "Description" ""
-			(at 67.31 119.38 0)
+			(at 67.31 134.62 0)
 			(effects
 				(font
@@
 			)
 		)
-		(property "Value" "500"
+		(property "Value" "150"
 			(at 78.74 69.8499 0)
 			(effects
@@
 			)
 		)
-		(property "Value" "180"
+		(property "Value" "100"
 			(at 53.34 96.52 90)
 			(effects
@@
 	(symbol
 		(lib_id "power:GND")
-		(at 63.5 130.81 0)
+		(at 63.5 146.05 0)
 		(unit 1)
 		(exclude_from_sim no)
@@
 		(fields_autoplaced yes)
 		(property "Reference" "#PWR09"
-			(at 63.5 137.16 0)
+			(at 63.5 152.4 0)
 			(effects
 				(font
@@
 		)
 		(property "Value" "GND"
-			(at 63.5 135.89 0)
+			(at 63.5 151.13 0)
 			(effects
 				(font
@@
 		)
 		(property "Footprint" ""
-			(at 63.5 130.81 0)
+			(at 63.5 146.05 0)
 			(effects
 				(font
@@
 		)
 		(property "Datasheet" ""
-			(at 63.5 130.81 0)
+			(at 63.5 146.05 0)
 			(effects
 				(font
@@
 		)
 		(property "Description" "Power symbol creates a global label with name \"GND\" , ground"
-			(at 63.5 130.81 0)
-			(effects
-				(font
+			(at 63.5 146.05 0)
+			(effects
+				(font
