File: Урок 8/ДЗ 8/ДЗ 8/ДЗ 8.kicad_sch (KiCad schematic)
At the start: 30 parts, among them K1 HONGFA_HFD2-0xx-x-L2-x, K2 HONGFA_HFD2-0xx-x-L2-x, SW1 SW_Push, SW2 SW_Push

Commit message: 1
Parts:
- R10: value 500 -> 10k
- R8: value 8 -> 500
Connections:
- net 12V: now also C2.1, C4.1, D2.1, D7.1; no longer R4.2, R9.2
- net GND: now also C1.1, C3.1, D2.2, D7.2, R4.2, R8.2
- net at D4.2 (A), D6.1 (K), K2.B1: now also Q3.1 (C); no longer C3.1, D7.2
- net at Q3.2 (B): now also R9.1; no longer R8.1
- net at R7.1, U3.4 (Collector): now also R9.2; no longer R8.2
- net at Q3.3 (A): now also R10.1; no longer R9.1
- net at D3.2 (A), D5.1 (K), K1.B1: now also Q2.1 (C); no longer C1.1, D2.2
- net at D4.1 (K): now also R8.1; no longer R10.1
Other:
- moved on the sheet: C1, C2, D2, D3, D5, K1, LA1, Q2, R1, R2, R3, R4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

Commit message: 1
Parts:
- removed C1, C3: 0.1uF, 564R60GAD10, symbol My_lib2:564R60GAD10
- removed C2, C4: 0.33uF, 564R60GAD10, symbol My_lib2:564R60GAD10
- removed D6: 1N4007, Diode_THT:D_DO-41_SOD81_P10.16mm_Horizontal, symbol Diode:1N4007
- removed D7: ~, My_lib2:TO-220 - L7805ACV, symbol My_lib2:L7805ACV
- removed Q3: ~, cadstarpcblib:BC32725PBFREE, symbol My_lib2:BC327-25_PBFREE
- removed R1, R2, R6, R7: 180, symbol Device:R
- removed R10, R3, R4, R9: 10k, symbol Device:R
- removed R5, R8: 500, symbol Device:R
- removed U3: ~, My_lib2:DIP762W60P254L460H450Q4N, symbol My_lib2:PC817X3NSZ9F
- added C1, C3: 0.33uF, My_lib2:564R60GAD10, symbol My_lib2:C_564R60GAD10
- added C2, C4: 0.1uF, My_lib2:564R60GAD10, symbol My_lib2:C_564R60GAD10
- added D3: 1N4007, Diode_THT:D_DO-41_SOD81_P10.16mm_Horizontal, symbol Diode:1N4007
- added J1, J2: ~, My_lib2:TB-09A, symbol My_lib2:TB-09A
- added Q2: ~, My_lib2:BC32725PBFREE, symbol My_lib2:BC327-25_PBFREE
- added R1, R10, R11, R12, R2, R3, R4, R5, R6, R7, R8, R9: ~, My_lib2:R, symbol My_lib2:R_CF100-3K3-J-TB-070-62
- added U2: ~, My_lib2:DIP762W60P254L460H450Q4N, symbol My_lib2:PC817X3NSZ9F
- added U4: ~, My_lib2:TO-220 - L7805ACV, symbol My_lib2:L7805ACV
- Q1: renamed from Q2; footprint cadstarpcblib:BC32725PBFREE -> My_lib2:BC32725PBFREE
- renumbered D5 to D1, D3 to D2, U2 to U1, D2 to U3
Connections:
- net 12V: now also J2.1, R12.1, R3.2, R6.1, R8.2; no longer U3.1
- net 3.3V: now also J1.1
- net GND: now also C1.2, C2.1, C2.2, C3.2, C4.1, C4.2, D3.2 (A), J1.2, J2.2, R10.2, R11.1, R4.2, R5.1, U2.2 (Cathode), U2.3 (Emitter), U4.2, U4.3 (GND)
- net at D4.2 (A), K2.B1: now also D3.1 (K), Q2.1 (C)
- net at D4.1 (K): now also R10.1
- net at SW2.2: now also R7.1
- net at SW1.2: now also R1.1
- net at U1.1 (Anode): now also R1.2
- net at D2.1 (K): now also R4.1
- net at Q1.2 (B): now also R2.2
- net at U1.4 (Collector): now also R2.1, R3.1
- net at Q1.3 (A): now also R5.2
- new net: C1.1, R6.2, U3.1
- new net: R8.1, R9.1, U2.4 (Collector)
- new net: C3.1, R12.2, U4.1
- new net: Q2.3 (A), R11.2
- new net: R7.2, U2.1 (Anode)
- new net: Q2.2 (B), R9.2
- no-connect marks 0 -> 5
Other:
- moved on the sheet: U3

Commit message: 1
Connections:
- net 12V: now also K1.11, K2.11
- removed net +12V: K1.11, K1.21, K2.11, K2.21
- no-connect marks 5 -> 12
Other:
- moved on the sheet: C3, C4, R11, R12, U4
