File: Урок 8/ДЗ 8/ДЗ 8/ДЗ 8.kicad_pcb (KiCad board)
At the start: 2 copper layers, 16 parts, among them K1 HONGFA_HFD2-0xx-x-L2-x, K2 HONGFA_HFD2-0xx-x-L2-x, SW1 SW_Push, SW2 SW_Push

Commit message: 1
Parts:
- added Q2: ~, My_lib2:BC32725PBFREE, F.Cu at (193.6, 86.8)
- added Q3: ~, My_lib2:BC32725PBFREE, F.Cu at (193.6, 93.5)
- added R1: ~, My_lib2:R, F.Cu at (148.6, 63.1)
- added R10: ~, My_lib2:R, F.Cu at (148.6, 100.4)
- added R11: ~, My_lib2:R, F.Cu at (148.6, 104.6)
- added R12: ~, My_lib2:R, F.Cu at (148.6, 108.7)
- added R2: ~, My_lib2:R, F.Cu at (148.6, 67.2)
- added R3: ~, My_lib2:R, F.Cu at (148.6, 71.4)
- added R4: ~, My_lib2:R, F.Cu at (148.6, 75.5)
- added R5: ~, My_lib2:R, F.Cu at (148.6, 79.7)
- added R6: ~, My_lib2:R, F.Cu at (148.6, 83.8)
- added R7: ~, My_lib2:R, F.Cu at (148.6, 88.0)
- added R8: ~, My_lib2:R, F.Cu at (148.6, 92.1)
- added R9: ~, My_lib2:R, F.Cu at (148.6, 96.3)
- C1, C3: value 0.1uF -> 0.33uF
- C2, C4: value 0.33uF -> 0.1uF
- moved SW2 59.9 mm to (185.8, 95.0)
- moved D3 59.9 mm to (200.5, 85.6)
- moved D4 59.9 mm to (200.5, 91.1)
- moved C1 59.6 mm to (169.0, 63.7)
- moved C2 59.6 mm to (169.0, 73.9)
- moved C3 59.6 mm to (169.0, 84.0)
- moved C4 59.6 mm to (169.0, 94.2)
- moved K1 59.6 mm to (182.8, 63.2)
- moved SW1 59.4 mm to (185.8, 86.9)
- moved D2 50.6 mm to (194.9, 102.8)
- moved U2 50.6 mm to (186.1, 102.3)
- moved U3 50.0 mm to (186.1, 109.0)
- moved D7 34.8 mm to (194.9, 109.0)
- moved D5 31.1 mm to (168.6, 103.7)
- moved D6 23.4 mm to (168.6, 107.9)
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Connections:
- C1 pad 1: Net-(D3-A) -> Net-(C1-Pad1)
- C2 pad 1: Net-(Q2-C) -> GND
- C3 pad 1: Net-(D4-A) -> Net-(C3-Pad1)
- C4 pad 1: Net-(Q3-C) -> GND
- D2 pad 1: Net-(Q2-C) -> Net-(C1-Pad1)
- D2 pad 2: Net-(D3-A) -> GND
- D7 pad 1: Net-(Q3-C) -> Net-(C3-Pad1)
- D7 pad 2: Net-(D4-A) -> GND

Commit message: 1
Parts:
- removed D5, D6: 1N4007, Diode_THT:D_DO-41_SOD81_P10.16mm_Horizontal
- removed D7: ~, My_lib2:TO-220 - L7805ACV
- removed Q3: ~, My_lib2:BC32725PBFREE
- added D1: 1N4007, Diode_THT:D_DO-41_SOD81_P10.16mm_Horizontal, F.Cu at (135.6, 100.7)
- added J1: ~, My_lib2:TB-09A, F.Cu at (114.0, 54.0)
- added J2: ~, My_lib2:TB-09A, F.Cu at (122.5, 54.0)
- added Q1: ~, My_lib2:BC32725PBFREE, F.Cu at (123.5, 67.0)
- added U1: ~, My_lib2:DIP762W60P254L460H450Q4N, F.Cu at (115.0, 86.0)
- added U4: ~, My_lib2:TO-220 - L7805ACV, F.Cu at (144.2, 78.0)
- D2: value ~ -> IR204A; footprint My_lib2:TO-220 - L7805ACV -> LED_THT:LED_D3.0mm_IRBlack
- D3: value IR204A -> 1N4007; footprint LED_THT:LED_D3.0mm_IRBlack -> Diode_THT:D_DO-41_SOD81_P10.16mm_Horizontal
- U3: footprint My_lib2:DIP762W60P254L460H450Q4N -> My_lib2:TO-220 - L7805ACV
- moved U3 79.4 mm to (129.4, 53.5)
- moved SW1 73.9 mm to (115.0, 66.0)
- moved D3 67.7 mm to (135.6, 104.9)
- moved C2 57.9 mm to (115.2, 95.2), turned to -90 degrees
- moved R10 53.9 mm to (202.5, 99.1)
- moved R11 53.9 mm to (202.5, 103.2)
- moved R12 53.9 mm to (202.5, 107.4)
- moved R4 53.9 mm to (202.5, 74.2)
- moved R5 53.9 mm to (202.5, 78.3)
- moved R6 53.9 mm to (202.5, 82.5)
- moved R7 53.9 mm to (202.5, 86.7)
- moved R8 53.9 mm to (202.5, 90.8)
- moved R9 53.9 mm to (202.5, 95.0)
- moved SW2 49.9 mm to (144.0, 67.8)
- moved R2 37.6 mm to (115.5, 85.3), turned to 90 degrees
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Connections:
- C1 pad 1: Net-(C1-Pad1) -> 12V
- C2 pad 1: GND -> Net-(C2-Pad1)
- C3 pad 1: Net-(C3-Pad1) -> 12V
- C4 pad 1: GND -> Net-(C4-Pad1)
- D2 pad 1: Net-(C1-Pad1) -> Net-(D2-K)
- D2 pad 2: GND -> Net-(D1-K)
- D3 pad 2: Net-(D3-A) -> GND
- D4 pad 2: Net-(D4-A) -> Net-(D3-K)
- K1 pad 11: +12V -> unconnected-(K1-Pad11)
- K1 pad 14: Net-(LA1--) -> unconnected-(K1-Pad14)
- K1 pad 21: +12V -> unconnected-(K1-Pad21)
- K1 pad B1: Net-(D3-A) -> Net-(D1-K)
- K2 pad 11: +12V -> unconnected-(K2-Pad11)
- K2 pad 14: Net-(LA2--) -> unconnected-(K2-Pad14)
- K2 pad 21: +12V -> unconnected-(K2-Pad21)
- K2 pad B1: Net-(D4-A) -> Net-(D3-K)
- Q2 pad 1: Net-(D3-A) -> Net-(D3-K)
- R1 pad 2: Net-(U2-Anode) -> Net-(U1-Anode)
- R11 pad 1: GND -> Net-(C4-Pad1)
- R11 pad 2: Net-(Q3-A) -> Net-(Q2-A)
- R12 pad 1: 12V -> Net-(C4-Pad1)
- R12 pad 2: Net-(C3-Pad1) -> GND
- R2 pad 1: Net-(U2-Collector) -> Net-(U1-Collector)
- R2 pad 2: Net-(Q2-B) -> Net-(Q1-B)
- R3 pad 1: Net-(U2-Collector) -> Net-(U1-Collector)
- R4 pad 1: Net-(D3-K) -> Net-(D2-K)
- R5 pad 1: GND -> Net-(C2-Pad1)
- R5 pad 2: Net-(Q2-A) -> Net-(Q1-A)
- R6 pad 1: 12V -> Net-(C2-Pad1)
- R6 pad 2: Net-(C1-Pad1) -> GND
- R7 pad 2: Net-(U3-Anode) -> Net-(U2-Anode)
- R8 pad 1: Net-(U3-Collector) -> Net-(U2-Collector)
- R9 pad 1: Net-(U3-Collector) -> Net-(U2-Collector)
- R9 pad 2: Net-(Q3-B) -> Net-(Q2-B)
- SW1 pad 2: Net-(R1-Pad1) -> unconnected-(SW1-Pad2)
- SW1 pad 3: (no net) -> unconnected-(SW1-1-Pad3)
- SW1 pad 4: (no net) -> Net-(R1-Pad1)
- SW2 pad 2: Net-(R7-Pad1) -> unconnected-(SW2-Pad2)
- SW2 pad 3: (no net) -> unconnected-(SW2-1-Pad3)
- SW2 pad 4: (no net) -> Net-(R7-Pad1)
- U3 pad 1: Net-(U3-Anode) -> 12V
- U3 pad 2: GND -> Net-(C2-Pad1)
Routing:
- net 12V: track 0.00 -> 18.6 mm
- net 3.3V: track 0.00 -> 9.98 mm
- net Net-(R1-Pad1): track 0.00 -> 7.68 mm
- net Net-(U1-Anode): track 0.00 -> 4.19 mm
Other:
- board outline added: 70 x 70 mm

Commit message: 1
Parts:
- added J3: ~, My_lib2:TB-09A, F.Cu at (160.2, 42.8)
- added J4: ~, My_lib2:TB-09A, F.Cu at (168.7, 42.8)
- C3: value 0.33uF -> 0.1uF
- C4: value 0.1uF -> 0.33uF
- moved R6 72.6 mm to (134.9, 56.0), turned to -90 degrees
- moved R5 71.3 mm to (131.3, 73.8), turned to 90 degrees
- moved C2 41.8 mm to (138.2, 60.4), turned to 0 degrees
- moved K1 39.5 mm to (127.0, 80.8), turned to 90 degrees
- moved D1 33.9 mm to (123.0, 69.2), turned to -90 degrees
- moved C3 31.8 mm to (175.0, 102.3)
- moved C4 31.8 mm to (159.3, 112.9)
- moved D2 31.8 mm to (190.7, 104.4)
- moved D3 31.8 mm to (158.8, 126.7)
- moved D4 31.8 mm to (196.5, 112.5)
- moved Q2 31.8 mm to (183.8, 112.3)
- moved U2 31.8 mm to (176.4, 127.7)
- moved SW2 27.7 mm to (165.5, 85.2)
- moved U4 24.4 mm to (150.2, 54.3), turned to 0 degrees
- moved C1 17.3 mm to (127.9, 52.9)
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Connections:
- C3 pad 1: 12V -> Net-(C3-Pad1)
- C4 pad 1: Net-(C4-Pad1) -> 12V
- D1 pad 2: GND -> Net-(D1-A)
- D2 pad 2: Net-(D1-K) -> GND
- D3 pad 2: GND -> Net-(D3-A)
- D4 pad 2: Net-(D3-K) -> GND
- K1 pad 11: unconnected-(K1-Pad11) -> 12V
- K1 pad 14: unconnected-(K1-Pad14) -> Net-(J3-Pad2)
- K1 pad A1: GND -> unconnected-(K1-PadA1)
- K1 pad B2: unconnected-(K1-PadB2) -> Net-(D1-A)
- K2 pad 11: unconnected-(K2-Pad11) -> 12V
- K2 pad 14: unconnected-(K2-Pad14) -> Net-(J4-Pad2)
- K2 pad A1: GND -> unconnected-(K2-PadA1)
- K2 pad B2: unconnected-(K2-PadB2) -> Net-(D3-A)
- R10 pad 1: Net-(D4-K) -> Net-(C3-Pad1)
- R10 pad 2: GND -> Net-(Q2-A)
- R11 pad 1: Net-(C4-Pad1) -> Net-(C3-Pad1)
- R11 pad 2: Net-(Q2-A) -> GND
- R12 pad 1: Net-(C4-Pad1) -> Net-(D4-K)
- R12 pad 2: GND -> Net-(D3-A)
- R4 pad 2: GND -> Net-(D1-A)
- U4 pad 2: Net-(C4-Pad1) -> Net-(C3-Pad1)
Routing:
- net Net-(D1-K): track 0.00 -> 34.1 mm
- net 12V: track 18.6 -> 35.2 mm
- net Net-(C2-Pad1): track 0.00 -> 10.9 mm
- net Net-(Q1-B): track 0.00 -> 9.37 mm
- net Net-(Q1-A): track 0.00 -> 8.59 mm
- net Net-(U1-Collector): track 0.00 -> 7.25 mm
- net 3.3V: track 9.98 -> 7.73 mm

Commit message: 1
Routing:
- net Net-(D1-A): track 0.00 -> 9.11 mm
Changed lines of the file:
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@@
 			(layer "F.Fab")
+		)
+		(fp_text user "K"
+			(at 0 -2.1 270)
+			(layer "F.SilkS")
+			(effects
+				(font
+					(size 1 1)
+					(thickness 0.15)
+				)
+			)
 		)
 		(fp_text user "${REFERENCE}"
 			(at 5.47 0 90)
+			(layer "F.Fab")
+			(effects
+				(font
+					(size 1 1)
+					(thickness 0.15)
+				)
+			)
+		)
+		(fp_text user "K"
+			(at 0 -2.1 270)
 			(layer "F.Fab")
 			(effects
@@
 	)
 	(segment
+		(start 131 72.28)
+		(end 131 79.379706)
+		(width 0.2)
+		(layer "F.Cu")
+		(net 1)
+	)
+	(segment
+		(start 123 74.25)
+		(end 123 69.17)
+		(width 0.2)
+		(layer "F.Cu")
+		(net 1)
+	)
+	(segment
 		(start 123.49 64.77)
 		(end 131 72.28)
@@
 	)
 	(segment
-		(start 131 72.28)
-		(end 131 79.379706)
-		(width 0.2)
-		(layer "F.Cu")
-		(net 1)
-	)
-	(segment
-		(start 123 74.240294)
-		(end 123 69.17)
+		(start 129.56 80.81)
+		(end 123 74.25)
 		(width 0.2)
 		(layer "F.Cu")
@@
 	(segment
 		(start 129.569706 80.81)
-		(end 123 74.240294)
+		(end 129.56 80.81)
 		(width 0.2)
 		(layer "F.Cu")
@@
 		(net 32)
 	)
+	(segment
+		(start 123.429706 79.33)
+		(end 123 79.33)
+		(width 0.2)
+		(layer "B.Cu")
+		(net 34)
+	)
+	(segment
+		(start 129.569706 73.19)
+		(end 123.429706 79.33)
+		(width 0.2)
+		(layer "B.Cu")
+		(net 34)
+	)
 	(embedded_fonts no)

Commit message: 1
Parts:
- removed C3: 0.1uF, My_lib2:564R60GAD10
- removed C4: 0.33uF, My_lib2:564R60GAD10
- removed R11: ~, My_lib2:R
- removed U4: ~, My_lib2:TO-220 - L7805ACV
- moved R7 136.3 mm to (73.2, 43.5), turned to -90 degrees
- moved R8 129.5 mm to (83.0, 41.0), turned to 90 degrees
- moved U2 122.6 mm to (80.0, 52.0), turned to 90 degrees
- moved SW2 101.0 mm to (75.2, 40.0), turned to -90 degrees
- moved R10 80.6 mm to (122.0, 103.7)
- moved R4 80.6 mm to (122.0, 78.8)
- moved R9 80.6 mm to (122.0, 99.5)
- moved R12 80.5 mm to (122.0, 107.8)
- moved R3 69.7 mm to (63.0, 41.5)
- moved SW1 64.4 mm to (55.0, 40.0), turned to -90 degrees
- moved J1 63.9 mm to (55.0, 30.0), turned to 180 degrees
- moved U1 63.5 mm to (60.0, 52.0), turned to 90 degrees
- moved R1 62.8 mm to (53.0, 43.5)
- moved D1 55.9 mm to (160.3, 110.8), turned to 0 degrees
- moved J4 55.0 mm to (115.2, 30.0)
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Connections:
- C2 pad 1: Net-(C2-Pad1) -> +5V
- R10 pad 1: Net-(C3-Pad1) -> +5V
- R5 pad 1: Net-(C2-Pad1) -> +5V
- R6 pad 1: Net-(C2-Pad1) -> +5V
- U3 pad 2: Net-(C2-Pad1) -> +5V
Routing:
- net Net-(D1-K): track 34.1 -> 0.00 mm
- net 12V: track 35.2 -> 7.08 mm
- net Net-(C2-Pad1): track 10.9 -> 0.00 mm
- net Net-(Q1-B): track 9.37 -> 0.00 mm
- net Net-(D1-A): track 9.11 -> 0.00 mm
- net Net-(Q1-A): track 8.59 -> 0.00 mm
- net Net-(R1-Pad1): track 7.68 -> 0.00 mm
- net Net-(U1-Collector): track 7.25 -> 0.00 mm
- net Net-(U1-Anode): track 4.19 -> 0.00 mm
- net 3.3V: track 7.73 -> 6.98 mm

Commit message: 1
Parts:
- moved R2 64.2 mm to (59.0, 58.5), turned to -90 degrees
Changed lines of the file:
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@@
 	(footprint "My_lib2:R"
 		(layer "F.Cu")
-		(at 121.985 70.48)
+		(at 58.95 58.4925 -90)
 		(property "Reference" "R2"
-			(at 8.7 -2.625 0)
+			(at 8.7 -2.625 270)
 			(unlocked yes)
 			(layer "F.SilkS")
@@
 		)
 		(property "Value" "~"
-			(at 2.54 1 0)
+			(at 2.54 1 270)
 			(unlocked yes)
 			(layer "F.Fab")
@@
 		)
 		(property "Datasheet" ""
-			(at 2.54 0 0)
+			(at 2.54 0 270)
 			(unlocked yes)
 			(layer "F.Fab")
@@
 		)
 		(property "Description" "CF100-3K3-J-TB-070-62 CARBON FILM FIXED RESISTOR, 1.0(1W)"
-			(at 2.54 0 0)
+			(at 2.54 0 270)
 			(unlocked yes)
 			(layer "F.Fab")
@@
 		)
 		(property "Description_1" "CARBON FILM FIXED RESISTOR, 1.0(1W)"
-			(at 0 0 0)
+			(at 0 0 270)
 			(unlocked yes)
 			(layer "F.Fab")
@@
 		)
 		(property "Height" ""
-			(at 0 0 0)
+			(at 0 0 270)
 			(unlocked yes)
 			(layer "F.Fab")
@@
 		)
 		(property "Manufacturer_Name" "HKR"
-			(at 0 0 0)
+			(at 0 0 270)
 			(unlocked yes)
 			(layer "F.Fab")
@@
 		)
 		(property "Manufacturer_Part_Number" "CF100-3K3-J-TB-070-62"
-			(at 0 0 0)
+			(at 0 0 270)
 			(unlocked yes)
 			(layer "F.Fab")
@@
 		)
 		(property "Mouser Part Number" ""
-			(at 0 0 0)
+			(at 0 0 270)
 			(unlocked yes)
 			(layer "F.Fab")
@@
 		)
 		(property "Mouser Price/Stock" ""
-			(at 0 0 0)
+			(at 0 0 270)
 			(unlocked yes)
 			(layer "F.Fab")
@@
 		)
 		(property "Arrow Part Number" ""
-			(at 0 0 0)
+			(at 0 0 270)
 			(unlocked yes)
 			(layer "F.Fab")
@@
 		)
 		(property "Arrow Price/Stock" ""
-			(at 0 0 0)
+			(at 0 0 270)
 			(unlocked yes)
 			(layer "F.Fab")
@@
 		(attr through_hole)
 		(fp_line
+			(start 5.65 1.15)
+			(end 5.65 -1.25)
+			(stroke
+				(width 0.2)
+				(type solid)
+			)
+			(layer "F.SilkS")
+		)
+		(fp_line
+			(start 11.95 1.15)
+			(end 5.65 1.15)
+			(stroke
+				(width 0.2)
+				(type solid)
+			)
+			(layer "F.SilkS")
+		)
+		(fp_line
 			(start 5.65 -1.25)
 			(end 11.95 -1.25)
@@
 		)
 		(fp_line
+			(start 11.95 -1.25)
+			(end 11.95 1.15)
+			(stroke
+				(width 0.2)
+				(type solid)
+			)
+			(layer "F.SilkS")
+		)
+		(fp_line
+			(start 2.54 1.5)
+			(end 2.54 -1.6)
+			(stroke
+				(width 0.05)
+				(type solid)
+			)
+			(layer "F.CrtYd")
+		)
+		(fp_line
+			(start 15.24 1.5)
+			(end 2.54 1.5)
+			(stroke
+				(width 0.05)
+				(type solid)
+			)
+			(layer "F.CrtYd")
+		)
+		(fp_line
+			(start 2.54 -1.6)
+			(end 15.24 -1.6)
+			(stroke
+				(width 0.05)
+				(type solid)
+			)
+			(layer "F.CrtYd")
+		)
+		(fp_line
+			(start 15.24 -1.6)
+			(end 15.24 1.5)
+			(stroke
+				(width 0.05)
+				(type solid)
+			)
+			(layer "F.CrtYd")
+		)
+		(fp_line
 			(start 5.65 1.15)
 			(end 5.65 -1.25)
 			(stroke
-				(width 0.2)
-				(type solid)
-			)
-			(layer "F.SilkS")
+				(width 0.1)
+				(type solid)
+			)
+			(layer "F.Fab")
+		)
+		(fp_line
+			(start 11.95 1.15)
+			(end 5.65 1.15)
+			(stroke
+				(width 0.1)
+				(type solid)
+			)
+			(layer "F.Fab")
+		)
+		(fp_line
+			(start 5.65 -1.25)
+			(end 11.95 -1.25)
+			(stroke
+				(width 0.1)
+				(type solid)
+			)
+			(layer "F.Fab")
 		)
 		(fp_line
@@
 			(end 11.95 1.15)
 			(stroke
-				(width 0.2)
-				(type solid)
-			)
-			(layer "F.SilkS")
-		)
-		(fp_line
-			(start 11.95 1.15)
-			(end 5.65 1.15)
-			(stroke
-				(width 0.2)
-				(type solid)
-			)
-			(layer "F.SilkS")
-		)
-		(fp_line
-			(start 2.54 -1.6)
-			(end 15.24 -1.6)
-			(stroke
-				(width 0.05)
-				(type solid)
-			)
-			(layer "F.CrtYd")
-		)
-		(fp_line
-			(start 2.54 1.5)
-			(end 2.54 -1.6)
-			(stroke
-				(width 0.05)
-				(type solid)
-			)
-			(layer "F.CrtYd")
-		)
-		(fp_line
-			(start 15.24 -1.6)
-			(end 15.24 1.5)
-			(stroke
-				(width 0.05)
-				(type solid)
-			)
-			(layer "F.CrtYd")
-		)
-		(fp_line
-			(start 15.24 1.5)
-			(end 2.54 1.5)
-			(stroke
-				(width 0.05)
-				(type solid)
-			)
-			(layer "F.CrtYd")
-		)
-		(fp_line
-			(start 5.65 -1.25)
-			(end 11.95 -1.25)
-			(stroke
-				(width 0.1)
-				(type solid)
-			)
-			(layer "F.Fab")
-		)
-		(fp_line
-			(start 5.65 1.15)
-			(end 5.65 -1.25)
-			(stroke
-				(width 0.1)
-				(type solid)
-			)
-			(layer "F.Fab")
-		)
-		(fp_line
-			(start 11.95 -1.25)
-			(end 11.95 1.15)
-			(stroke
-				(width 0.1)
-				(type solid)
-			)
-			(layer "F.Fab")
-		)
-		(fp_line
-			(start 11.95 1.15)
-			(end 5.65 1.15)
-			(stroke
 				(width 0.1)
 				(type solid)
@@
 		)
 		(fp_text user "${REFERENCE}"
-			(at 0.85 -0.05 0)
+			(at 0.85 -0.05 90)
 			(layer "F.Fab")
 			(effects
@@
 		)
 		(pad "1" thru_hole circle
-			(at 4.2 -0.05)
+			(at 4.2 -0.05 270)
 			(size 1.2 1.2)
 			(drill 0.8)
@@
 		)
 		(pad "2" thru_hole circle
-			(at 13.4 0)
+			(at 13.4 0 270)
 			(size 1.2 1.2)
 			(drill 0.8)

Commit message: 1
Parts:
- R1, R7: value ~ -> 100
- R10, R5: value ~ -> 47
- R12, R3, R4, R8: value ~ -> 510
- R2, R9: value ~ -> 1000
Connections:
- D2 pad 1: Net-(D2-K) -> GND
- D2 pad 2: GND -> Net-(D2-A)
- D4 pad 1: Net-(D4-K) -> GND
- D4 pad 2: GND -> Net-(D4-A)
- R12 pad 1: Net-(D4-K) -> Net-(D4-A)
- R4 pad 1: Net-(D2-K) -> Net-(D2-A)
Changed lines of the file:
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@@
 	(net 1 "Net-(D1-K)")
 	(net 2 "GND")
-	(net 3 "Net-(D2-K)")
+	(net 3 "Net-(D2-A)")
 	(net 4 "Net-(D3-K)")
-	(net 5 "Net-(D4-K)")
+	(net 5 "Net-(D4-A)")
 	(net 6 "unconnected-(K1-Pad24)")
 	(net 7 "unconnected-(K1-Pad22)")
@@
 			(remove_unused_layers no)
 			(net 12 "unconnected-(K2-Pad12)")
-			(pintype "passive")
+			(pintype "passive+no_connect")
 		)
 		(pad "14" thru_hole circle
@@
 			(roundrect_rratio 0.125)
 			(net 38 "unconnected-(K2-PadA1)")
-			(pintype "passive")
+			(pintype "passive+no_connect")
 		)
 		(pad "A2" thru_hole circle
@@
 			(layers "*.Cu" "*.Mask")
 			(remove_unused_layers no)
-			(net 3 "Net-(D2-K)")
+			(net 2 "GND")
 			(pinfunction "K")
 			(pintype "passive")
@@
 			(layers "*.Cu" "*.Mask")
 			(remove_unused_layers no)
-			(net 2 "GND")
+			(net 3 "Net-(D2-A)")
 			(pinfunction "A")
 			(pintype "passive")
@@
 			)
 		)
-		(property "Value" "~"
+		(property "Value" "100"
 			(at 2.54 1 270)
 			(unlocked yes)
@@
 			)
 		)
-		(property "Value" "~"
+		(property "Value" "1000"
 			(at 2.54 1 0)
 			(unlocked yes)
@@
 			)
 		)
-		(property "Value" "~"
+		(property "Value" "510"
 			(at 2.54 1 90)
 			(unlocked yes)
@@
 			)
 		)
-		(property "Value" "~"
+		(property "Value" "47"
 			(at 2.54 1 0)
 			(unlocked yes)
@@
 			)
 		)
-		(property "Value" "~"
+		(property "Value" "47"
 			(at 2.54 1 0)
 			(unlocked yes)
@@
 			)
 		)
-		(property "Value" "~"
+		(property "Value" "100"
 			(at 2.54 1 270)
 			(unlocked yes)
@@
 	)
 	(footprint "My_lib2:TB-09A"
+		(locked yes)
 		(layer "F.Cu")
 		(at 55 30 180)
@@
 			)
 		)
-		(property "Value" "~"
+		(property "Value" "510"
 			(at 2.54 1 90)
 			(unlocked yes)
@@
 			(remove_unused_layers no)
 			(net 10 "unconnected-(K1-Pad12)")
-			(pintype "passive")
+			(pintype "passive+no_connect")
 		)
 		(pad "14" thru_hole circle
@@
 			(roundrect_rratio 0.125)
 			(net 37 "unconnected-(K1-PadA1)")
-			(pintype "passive")
+			(pintype "passive+no_connect")
 		)
 		(pad "A2" thru_hole circle
@@
 			)
 		)
-		(property "Value" "~"
+		(property "Value" "510"
 			(at 2.54 1 0)
 			(unlocked yes)
@@
 			(layers "*.Cu" "*.Mask")
 			(remove_unused_layers no)
-			(net 5 "Net-(D4-K)")
+			(net 5 "Net-(D4-A)")
 			(pintype "passive")
 		)
@@
 			)
 		)
-		(property "Value" "~"
+		(property "Value" "510"
 			(at 2.54 1 0)
 			(unlocked yes)
@@
 			(layers "*.Cu" "*.Mask")
 			(remove_unused_layers no)
-			(net 3 "Net-(D2-K)")
+			(net 3 "Net-(D2-A)")
 			(pintype "passive")
 		)
@@
 			)
 		)
-		(property "Value" "~"
+		(property "Value" "1000"
 			(at 2.54 1 270)
 			(unlocked yes)
@@
 			(layers "*.Cu" "*.Mask")
 			(remove_unused_layers no)
-			(net 5 "Net-(D4-K)")
+			(net 2 "GND")
 			(pinfunction "K")
 			(pintype "passive")
@@
 			(layers "*.Cu" "*.Mask")
 			(remove_unused_layers no)
-			(net 2 "GND")
+			(net 5 "Net-(D4-A)")
 			(pinfunction "A")
 			(pintype "passive")

Commit message: 1
Parts:
- removed R6: ~, My_lib2:R
- moved C1 107.3 mm to (77.2, 29.1)
- moved C2 106.6 mm to (77.2, 37.1)
- moved U3 106.6 mm to (71.2, 29.4), turned to -90 degrees
- moved D1 105.5 mm to (63.9, 68.0)
- moved Q1 103.6 mm to (60.0, 63.5), turned to 90 degrees
- moved D2 97.2 mm to (72.0, 90.0), turned to 90 degrees
- moved D3 93.1 mm to (79.9, 68.0)
- moved Q2 82.6 mm to (82.0, 61.3), turned to 90 degrees
- moved K1 81.8 mm to (58.2, 73.3)
- moved R10 80.2 mm to (73.8, 39.5), turned to -90 degrees
- moved D4 74.0 mm to (96.0, 90.0), turned to 90 degrees
- moved R9 73.0 mm to (80.5, 39.5), turned to -90 degrees
- moved K2 70.3 mm to (81.4, 74.3)
- moved R5 70.1 mm to (66.9, 39.5), turned to -90 degrees
- moved R4 50.7 mm to (72.0, 87.5), turned to 90 degrees
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Connections:
- U3 pad 2: +5V -> GND
- U3 pad 3: GND -> +5V
Routing:
- net 12V: track 7.08 -> 153.1 mm
- net Net-(J3-Pad2): track 0.00 -> 54.4 mm
- net 3.3V: track 6.98 -> 47.2 mm
- net Net-(U1-Collector): track 0.00 -> 29.5 mm
- net Net-(J4-Pad2): track 0.00 -> 28.1 mm
- net Net-(U2-Collector): track 0.00 -> 27.9 mm
- net +5V: track 0.00 -> 22.6 mm
- net Net-(D3-A): track 0.00 -> 19.6 mm
- net Net-(D1-A): track 0.00 -> 18.5 mm
- net Net-(D3-K): track 0.00 -> 17.3 mm
- net Net-(D1-K): track 0.00 -> 16.5 mm
- net Net-(Q1-B): track 0.00 -> 12.0 mm
- net Net-(Q1-A): track 0.00 -> 10.8 mm
- net Net-(Q2-A): track 0.00 -> 10.6 mm
- net Net-(Q2-B): track 0.00 -> 7.22 mm
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- added copper zone on B.Cu, net GND
- added copper zone on F.Cu, net GND
Other:
- board size 70 x 70 mm -> 63.5 x 70.5 mm
