File: Урок 9/9 лекция/ДЗ 9/9/_autosave-9.kicad_sch (KiCad schematic)
At the start: 11 parts, among them IC1 LM393P, SW1 SW_Push

Commit message: 1
Parts:
- removed C1: ~, My_lib2:564R60GAD10, symbol My_lib2:C_564R60GAD10
- added C2: ~, My_lib2:C - 564R60GAD10, symbol My_lib2:C_564R60GAD10
- C1: renamed from C2; footprint My_lib2:564R60GAD10 -> My_lib2:C - 564R60GAD10
- R1, R2, R3, R4, R5: footprint My_lib2:R -> My_lib2:R axil
- SW1: footprint My_lib2:0650HIM-130G-G -> My_lib2:SW - 0650HIM-130G-G
Connections:
- net 9V: now also C2.1; no longer C1.2
- net GND: now also C1.2, C2.2; no longer C1.1
- net at D1.3, R1.2: now also C1.1
Other:
- moved on the sheet: C1
