File: Урок 9/9 лекция/ДЗ 9/9/9.kicad_sch (KiCad schematic)
At the start: 6 parts

Commit message: R9
Parts:
- added C3: ~, My_lib2:C - 564R60GAD10, symbol My_lib2:C_564R60GAD10
- added D2: 1N5711, Diode_THT:D_DO-35_SOD27_P7.62mm_Horizontal, symbol Diode:1N5711
- added IC1, IC2: ~, My_lib2:8-DIP, symbol My_lib2:NE555
- added IC1: LM393P, My_lib2:8-DIP, symbol My_lib2:LM393P
- added R3, R4, R5, R6, R7, R8: ~, My_lib2:R axil, symbol My_lib2:R_CF100-3K3-J-TB-070-62
- added SW1: SW_Push, My_lib2:SW - 0650HIM-130G-G, symbol My_lib2:SW_Push
- C1, C2: footprint My_lib2:564R60GAD10 -> My_lib2:C - 564R60GAD10
- D1: footprint My_liblary:TO-220 - L7805ACV -> My_lib2:TO-220 - L7805ACV
- R1, R2: footprint My_lib2:R -> My_lib2:R axil
Connections:
- net GND: now also C1.2, C2.2, J1.2, C3.2, IC1.1, IC1.4 (GND), R3.1, R5.2, R7.1; no longer C1.1, C2.1, R2.1
- net at D1.1, R2.2: now also R3.2; no longer R1.1
- new net: D2.1 (K), IC1.2, IC1.6, R6.1, R7.2
- new net: C3.1, D2.2 (A), R8.2
- new net: J1.1, R1.1
- new net: C1.1, D1.3, R1.2
- new net: IC1.7 (2OUT), R8.1
- new net: IC1.5 (2IN+), SW1.4 (2)
- new net 2IN- - IC1: IC1.6 (2IN-), R4.2, R5.1
- new net 9V: C2.1, D1.2, IC1.4, IC1.8, IC1.8 (VCC), R2.1, R4.1, R6.2
- new net OUT - NE555: IC1.3, SW1.1
- no-connect marks 0 -> 7
