File: Урок 9/9 лекция/ДЗ 9/9/9.kicad_sch (KiCad schematic)
At the start: 18 parts, among them IC1 LM393P, SW1 SW_Push

Commit message: R9
Parts:
- added C4: ~, My_lib2:C - 564R60GAD10, symbol My_lib2:C_564R60GAD10
- added D3: LED, symbol Device:LED
- added R10, R11, R9: ~, My_lib2:R axil, symbol My_lib2:R_CF100-3K3-J-TB-070-62
Connections:
- net GND: now also IC2.1, C4.2, D3.1 (K)
- net OUT - NE555: now also IC2.4, IC2.8, R9.2
- net at IC2.2: now also IC2.6, C4.1, R10.1
- net at IC2.3: now also R11.2
- net at IC2.7: now also R10.2, R9.1
- net 2IN- - IC1: no longer names the net of IC1.6 (2IN-), R4.2, R5.1
- new net: D3.2 (A), R11.1
- no-connect marks 7 -> 8
Other:
- moved on the sheet: IC2

Commit message: r9
Parts:
- added D4: LED, symbol Device:LED
- added R12: 500, My_lib2:R axil, symbol My_lib2:R_CF100-3K3-J-TB-070-62
- C1: value ~ -> 0.33uF
- C2: value ~ -> 0.1uF
- C3: value ~ -> 0.47uF
- C4: value ~ -> 1uF
- D2: value 1N5711 -> 1N5819
- R1: value ~ -> 40
- R10: value ~ -> 1M
- R11: value ~ -> 500
- R2: value ~ -> 100
- R3: value ~ -> 620
- R4, R6, R7, R9: value ~ -> 1000
- R5: value ~ -> 2000
- R8: value ~ -> 100k
Connections:
- net GND: now also D4.1 (K)
- net OUT - NE555: now also R12.2
- new net: D4.2 (A), R12.1
Other:
- moved on the sheet: C2, D3, R1, R11

Commit message: Финал
Parts:
- removed D2: 1N5819, Diode_THT:D_DO-35_SOD27_P7.62mm_Horizontal, symbol Diode:1N5711
- removed IC1: LM393P, My_lib2:8-DIP, symbol My_lib2:LM393P
- removed R4: 1000, My_lib2:R axil, symbol My_lib2:R_CF100-3K3-J-TB-070-62
- removed R5: 2000, My_lib2:R axil, symbol My_lib2:R_CF100-3K3-J-TB-070-62
Connections:
- net OUT - NE555: now also R8.1; no longer SW1.1
- net at IC1.2, IC1.6, R6.1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: now also SW1.1
- net at C3.1, R8.2: now also SW1.4 (2)
- no-connect marks 8 -> 5
Other:
- moved on the sheet: C3, D4, R12, R8, SW1
