File: Урок 9/9 лекция/ДЗ 9/9.kicad_sch (KiCad schematic)
At the start: 18 parts, among them IC1 LM393P, SW1 SW_Push

Commit message: 10
Parts:
- removed D2: 1N5711, Diode_THT:D_DO-35_SOD27_P7.62mm_Horizontal, symbol Diode:1N5711
- removed IC1: LM393P, My_lib2:8-DIP, symbol My_lib2:LM393P
- removed R4, R5: ~, My_lib2:R axil, symbol My_lib2:R_CF100-3K3-J-TB-070-62
- added C4: 1uF, My_lib2:C - 564R60GAD10, symbol My_lib2:C_564R60GAD10
- added D3, D4: LED, symbol Device:LED
- added R10: 1M, My_lib2:R axil, symbol My_lib2:R_CF100-3K3-J-TB-070-62
- added R11, R12: 500, My_lib2:R axil, symbol My_lib2:R_CF100-3K3-J-TB-070-62
- added R9: 1000, My_lib2:R axil, symbol My_lib2:R_CF100-3K3-J-TB-070-62
- C1: value ~ -> 0.33uF
- C2: value ~ -> 0.1uF
- C3: value ~ -> 0.47uF
- R1: value ~ -> 40
- R2: value ~ -> 100
- R3: value ~ -> 620
- R6, R7: value ~ -> 1000
- R8: value ~ -> 100k
Connections:
- net 9V: now also R1.2; no longer D1.2, R2.1
- net GND: now also IC2.1, IC2.3, C4.2, D4.1 (K), R11.2
- net OUT - NE555: now also IC2.4, IC2.8, R8.1, R12.2, R9.2; no longer SW1.1
- net at IC1.2, IC1.6, R6.1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: now also SW1.1
- net at C3.1, R8.2: now also SW1.4 (2)
- net at J1.1: now also C1.1, D1.3; no longer R1.1
- net at IC2.2: now also IC2.6, C4.1, R10.1
- net at IC2.7: now also R10.2, R9.1
- new net: D3.2 (A), R11.1
- new net: D4.2 (A), R12.1
- new net: D1.2, R1.1, R2.1
- no-connect marks 7 -> 5
Other:
- moved on the sheet: C2, C3, IC2, J1, R1, R2, R8, SW1

Commit message: hom
Connections:
- net GND: now also D3.1 (K); no longer IC2.3, R11.2
- new net: IC2.3, R11.2
Changed lines of the file:
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@@
+	)
+	(junction
+		(at 74.93 147.32)
+		(diameter 0)
+		(color 0 0 0 0)
 	)
 	(junction
@@
 	)
 	(junction
-		(at 74.93 147.32)
-		(diameter 0)
-		(color 0 0 0 0)
-	)
-	(junction
 		(at 54.61 50.8)
 		(diameter 0)
@@
 	(junction
 		(at 33.02 130.81)
-		(diameter 0)
-		(color 0 0 0 0)
-	)
-	(junction
-		(at 87.63 93.98)
 		(diameter 0)
 		(color 0 0 0 0)
@@
 	(wire
 		(pts
-			(xy 74.93 147.32) (xy 101.6 147.32)
-		)
-		(stroke
-			(width 0)
-			(type default)
-		)
-	)
-	(wire
-		(pts
 			(xy 154.94 40.64) (xy 157.48 40.64)
 		)
@@
 	(wire
 		(pts
-			(xy 101.6 93.98) (xy 101.6 147.32)
-		)
-		(stroke
-			(width 0)
-			(type default)
-		)
-	)
-	(wire
-		(pts
 			(xy 34.29 43.18) (xy 34.29 33.02)
 		)
@@
 	(wire
 		(pts
+			(xy 87.63 147.32) (xy 74.93 147.32)
+		)
+		(stroke
+			(width 0)
+			(type default)
+		)
+	)
+	(wire
+		(pts
 			(xy 133.35 55.88) (xy 142.24 55.88)
 		)
@@
 	(wire
 		(pts
+			(xy 87.63 121.92) (xy 87.63 147.32)
+		)
+		(stroke
+			(width 0)
+			(type default)
+		)
+	)
+	(wire
+		(pts
 			(xy 157.48 40.64) (xy 160.02 40.64)
 		)
@@
 		)
 		(stroke
-			(width 0)
-			(type default)
-		)
-	)
-	(wire
-		(pts
-			(xy 87.63 93.98) (xy 101.6 93.98)
-		)
-		(stroke
