File: Урок 14/ДЗ/14/14.kicad_sch (KiCad schematic)
At the start: 13 parts, among them U1 STM32G473RETx

Commit message: 14
Parts:
- added C11, C14: 0.1uF, My_lib2:564R60GAD10, symbol My_Lib:C - 564R60GAD10
- added C12: 1uF, My_lib2:564R60GAD10, symbol My_Lib:C - 564R60GAD10
- added C13: 47pF, My_lib2:564R60GAD10, symbol My_Lib:C - 564R60GAD10
- added D1: ~, symbol Device:D_Schottky
- added FB1: 600Ом 100Мгц, symbol Device:FerriteBead
- added J2: ~, symbol My_Lib:J - B4P-VH
- added R1, R2: 100, RESAD2700W60L1100D400, symbol My_Lib:R - CF100-3K3-J-TB-070-62
- added R3: 1k, RESAD2700W60L1100D400, symbol My_Lib:R - CF100-3K3-J-TB-070-62
- added R4: 10k, RESAD2700W60L1100D400, symbol My_Lib:R - CF100-3K3-J-TB-070-62
- added SW1: SW_Push, My_lib2:0650HIM-130G-G, symbol My_Lib:SW_Push
- C1: value 0.1uF -> 0.33uF
Connections:
- net 3.3V: now also FB1.2, R3.2, R4.2; no longer U1.29 (VDDA)
- net GND: now also C11.1, C12.1, C13.1, C14.1, J2.4, SW1.1
- net at U1.49 (PA13): now also R1.1
- net at U1.50 (PA14): now also C13.2, R2.1
- net RESET: now reaches U1.7 (PG10)
- net RESET: now also C14.2, R4.1, SW1.2
- net at C1.2, U2.1 (IN), U2.3 (GND): now also D1.1 (K); no longer J1.2
- new net: J2.2, R1.2
- new net: D1.2 (A), J1.2
- new net: J2.1, R3.1
- new net: J2.3, R2.2
- new net 3.3VA: C11.2, C12.2, FB1.1, U1.29 (VDDA)
Other:
- note added: "SWCLK"
- note added: "SWDIO"
