File: Урок 14/ДЗ/14/14.kicad_pcb (KiCad board)
At the start: 2 copper layers, 61.4 x 24.7 mm, 26 parts, among them SW1 SW_Push, U1 STM32G473RETx

Commit message: 14
Parts:
- SW1: footprint My_lib2:0650HIM-130G-G -> My_lib2:SW - 0650HIM-130G-G
- moved SW1 0.15 mm to (67.1, 64.2)
Routing:
- net GND: track 1.78 -> 1.26 mm, vias 7 -> 10
Changed lines of the file:
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@@
 	)
 	(setup
+		(stackup
+			(layer "F.SilkS"
+				(type "Top Silk Screen")
+			)
+			(layer "F.Paste"
+				(type "Top Solder Paste")
+			)
+			(layer "F.Mask"
+				(type "Top Solder Mask")
+				(thickness 0.01)
+			)
+			(layer "F.Cu"
+				(type "copper")
+				(thickness 0.035)
+			)
+			(layer "dielectric 1"
+				(type "core")
+				(thickness 1.51)
+				(material "FR4")
+				(epsilon_r 4.5)
+				(loss_tangent 0.02)
+			)
+			(layer "B.Cu"
+				(type "copper")
+				(thickness 0.035)
+			)
+			(layer "B.Mask"
+				(type "Bottom Solder Mask")
+				(thickness 0.01)
+			)
+			(layer "B.Paste"
+				(type "Bottom Solder Paste")
+			)
+			(layer "B.SilkS"
+				(type "Bottom Silk Screen")
+			)
+			(copper_finish "None")
+			(dielectric_constraints no)
+		)
 		(pad_to_mask_clearance 0)
 		(allow_soldermask_bridges_in_footprints no)
@@
 	(net 61 "unconnected-(U1-PB14-Pad36)")
 	(net 62 "unconnected-(U2-NC-Pad4)")
-	(net 63 "unconnected-(SW1-Pad1)")
-	(net 64 "unconnected-(SW1-Pad4)")
+	(net 63 "unconnected-(SW1-Pad4)")
+	(net 64 "unconnected-(SW1-Pad1)")
 	(footprint "Resistor_SMD:R_0201_0603Metric"
 		(layer "F.Cu")
@@
 			(at 0 1.05 90)
 			(layer "F.Fab")
+			(hide yes)
 			(effects
 				(font
@@
 			(at 0 1.05 0)
 			(layer "F.Fab")
+			(hide yes)
 			(effects
 				(font
@@
 			(at 0 1.05 0)
 			(layer "F.Fab")
+			(hide yes)
 			(effects
 				(font
@@
 			(at -0.05 1.7 90)
 			(layer "F.Fab")
+			(hide yes)
 			(effects
 				(font
@@
 			(at 0 2.05 90)
 			(layer "F.Fab")
+			(hide yes)
 			(effects
 				(font
@@
 		)
 	)
-	(footprint "My_lib2:0650HIM-130G-G"
-		(layer "F.Cu")
-		(at 67.2 64.15)
-		(property "Reference" "SW1"
-			(at 0 -4.75 0)
-			(unlocked yes)
-			(layer "F.SilkS")
-			(effects
-				(font
-					(size 1 1)
-					(thickness 0.1)
-				)
-			)
-		)
-		(property "Value" "SW_Push"
-			(at -0.125 5.25 0)
-			(unlocked yes)
-			(layer "F.Fab")
-			(hide yes)
-			(effects
-				(font
-					(size 1 1)
-					(thickness 0.15)
-				)
-			)
-		)
-		(property "Datasheet" ""
-			(at 0 0 0)
-			(unlocked yes)
-			(layer "F.Fab")
-			(hide yes)
-			(effects
-				(font
-					(size 1 1)
-					(thickness 0.15)
-				)
-			)
-		)
-		(property "Description" "Push button switch, generic, two pins"
-			(at 0 0 0)
-			(unlocked yes)
-			(layer "F.Fab")
-			(hide yes)
-			(effects
-				(font
-					(size 1 1)
-					(thickness 0.15)
-				)
-			)
-		)
-		(sheetname "/")
-		(sheetfile "14.kicad_sch")
-		(attr through_hole)
-		(fp_rect
-			(start -2.25 -2.25)
-			(end 2.25 2.25)
-			(stroke
-				(width 0.1)
-				(type solid)
-			)
-			(fill no)
-			(layer "F.SilkS")
-		)
-		(fp_rect
-			(start -4.5 -3.5)
-			(end 4.5 3.5)
-			(stroke
-				(width 0.05)
-				(type solid)
-			)
-			(fill no)
-			(layer "F.CrtYd")
-		)
-		(pad "1" thru_hole rect
-			(at -3.25 -2.25)
-			(size 1.8 1.8)
-			(drill 1)
-			(layers "*.Cu" "*.Mask")
-			(remove_unused_layers no)
-			(net 63 "unconnected-(SW1-Pad1)")
-			(pinfunction "1")
-			(pintype "passive")
-		)
-		(pad "2" thru_hole circle
-			(at 3.25 -2.25)
-			(size 1.8 1.8)
-			(drill 1)
-			(layers "*.Cu" "*.Mask")
-			(remove_unused_layers no)
-			(net 5 "RESET")
-			(pintype "passive")
-		)
-		(pad "3" thru_hole circle
-			(at -3.25 2.25)
-			(size 1.8 1.8)
-			(drill 1)
-			(layers "*.Cu" "*.Mask")
-			(remove_unused_layers no)
-			(net 2 "GND")
-			(pintype "passive")
-		)
-		(pad "4" thru_hole circle
-			(at 3.25 2.25)
-			(size 1.8 1.8)
-			(drill 1)
-			(layers "*.Cu" "*.Mask")
-			(remove_unused_layers no)
-			(net 64 "unconnected-(SW1-Pad4)")
-			(pintype "passive")
-		)
-		(embedded_fonts no)
-	)
 	(footprint "Resistor_SMD:R_0805_2012Metric"
 		(layer "F.Cu")
@@
 			(at 0 1.65 0)
 			(layer "F.Fab")
+			(hide yes)
 			(effects
 				(font
@@
 		(embedded_fonts no)
 	)
+	(footprint "My_lib2:SW - 0650HIM-130G-G"
+		(layer "F.Cu")
+		(at 67.056 64.171)
+		(property "Reference" "SW1"
+			(at 0 -4.625 0)
+			(unlocked yes)
+			(layer "F.SilkS")
+			(effects
+				(font
+					(size 1 1)
+					(thickness 0.2)
+					(bold yes)
+				)
+			)
+		)
+		(property "Value" "SW_Push"
+			(at -0.125 5.25 0)
+			(unlocked yes)
+			(layer "F.Fab")
+			(hide yes)
+			(effects
+				(font
+					(size 1 1)
+					(thickness 0.15)
+				)
+			)
+		)
+		(property "Datasheet" ""
+			(at 0 0 0)
+			(unlocked yes)
+			(layer "F.Fab")
+			(hide yes)
+			(effects
+				(font
+					(size 1 1)
+					(thickness 0.15)
+				)
+			)
+		)
+		(property "Description" "Push button switch, generic, two pins"
+			(at 0 0 0)
+			(unlocked yes)
+			(layer "F.Fab")
+			(hide yes)
+			(effects
+				(font
+					(size 1 1)
+					(thickness 0.15)
+				)
+			)
+		)
+		(sheetname "/")
+		(sheetfile "14.kicad_sch")
+		(attr through_hole)
+		(fp_rect
+			(start -2.25 -2.25)
+			(end 2.25 2.25)
+			(stroke
+				(width 0.1)
+				(type solid)
+			)
+			(fill no)
+			(layer "F.SilkS")
+		)
+		(fp_rect
+			(start -4.5 -3.5)
+			(end 4.5 3.5)
+			(stroke
+				(width 0.05)
+				(type solid)
+			)
+			(fill no)
+			(layer "F.CrtYd")
+		)
+		(pad "1" thru_hole rect
+			(at -3.25 -2.25)
+			(size 1.8 1.8)
+			(drill 1)
+			(layers "*.Cu" "*.Mask")
+			(remove_unused_layers no)
+			(net 64 "unconnected-(SW1-Pad1)")
+			(pinfunction "1")
+			(pintype "passive+no_connect")
+		)
+		(pad "2" thru_hole circle
+			(at 3.25 -2.25)
+			(size 1.8 1.8)
+			(drill 1)
+			(layers "*.Cu" "*.Mask")
+			(remove_unused_layers no)
+			(net 5 "RESET")
+			(pintype "passive")
+		)
+		(pad "3" thru_hole circle
+			(at -3.25 2.25)
+			(size 1.8 1.8)
+			(drill 1)
+			(layers "*.Cu" "*.Mask")
+			(remove_unused_layers no)
+			(net 2 "GND")
+			(pintype "passive")
+		)
+		(pad "4" thru_hole circle
+			(at 3.25 2.25)
+			(size 1.8 1.8)
+			(drill 1)
+			(layers "*.Cu" "*.Mask")
+			(remove_unused_layers no)
+			(net 63 "unconnected-(SW1-Pad4)")
+			(pintype "passive+no_connect")
+		)
+		(embedded_fonts no)
+	)
 	(footprint "Resistor_SMD:R_0201_0603Metric"
 		(layer "F.Cu")
@@
 		(tags "SOD-123")
 		(property "Reference" "D1"
-			(at 0 -2 0)
+			(at -0.102 -2 0)
 			(layer "F.SilkS")
 			(effects
@@
 		)
 		(fp_text user "${REFERENCE}"
-			(at 0 -2 0)
+			(at 0 -2 180)
 			(layer "F.Fab")
 			(effects
@@
 	(gr_poly
 		(pts
-			(xy 74.35 55.525) (xy 75.425 55.525) (xy 75.425 54.175) (xy 74.35 54.2)
-		)
-		(stroke
-			(width 0.2)
-			(type solid)
-		)
-		(fill yes)
-		(layer "F.Cu")
-		(net 2)
-	)
-	(gr_poly
-		(pts
-			(xy 83.799473 69.174996) (xy 84.405588 69.179412) (xy 84.401537 69.37562) (xy 83.799473 69.375542)
-		)
-		(stroke
-			(width 0.2)
-			(type solid)
-		)
-		(fill yes)
-		(layer "F.Cu")
-		(net 2)
-	)
-	(gr_poly
-		(pts
 			(xy 88.145588 66.329412) (xy 87.645588 66.329412) (xy 87.645588 67.679412) (xy 88.145588 67.679412)
 		)
@@
 	)
 	(segment
-		(start 85.645588 65.745588)
-		(end 85.275 65.375)
-		(width 0.2)
-		(layer "F.Cu")
-		(net 2)
-	)
-	(segment
 		(start 85.645588 67.004412)
 		(end 85.645588 65.745588)
@@
 	)
 	(via
+		(at 85.915588 69.254528)
+		(size 0.6)
+		(drill 0.3)
+		(layers "F.Cu" "B.Cu")
+		(net 2)
+	)
+	(via
 		(at 80.95 53.825)
 		(size 0.6)
@@
 	)
 	(via
+		(at 88.519 69.977)
+		(size 0.6)
+		(drill 0.3)
+		(layers "F.Cu" "B.Cu")
+		(free yes)
+		(net 2)
+	)
+	(via
+		(at 87.65 52.85)
+		(size 0.6)
+		(drill 0.3)
+		(layers "F.Cu" "B.Cu")
+		(free yes)
+		(net 2)
+	)
+	(via
 		(at 66.65 54.975)
 		(size 0.6)
@@
 		(name "3.3V")
 		(hatch full 0.5)
-		(connect_pads yes
+		(connect_pads
 			(clearance 0.5)
 		)
@@
 		(hatch full 0.5)
 		(priority 1)
-		(connect_pads yes
+		(connect_pads
 			(clearance 0.5)
 		)
