File: Урок 15/ДЗ/15/15.kicad_pcb (KiCad board)
At the start: 2 copper layers, 41 parts, among them SW1 SW_Push, SW2 SW_Push, SW3 SW_Push, SW4 SW_Push, SW5 SW_Push, U3 STM32F103C8Tx, Y1 Crystal_GND24

Commit message: 15
Parts:
- moved C11 72.0 mm to (52.4, 46.0), turned to -90 degrees
- moved FB1 71.5 mm to (55.3, 48.2), turned to -90 degrees
- moved C12 71.2 mm to (53.7, 48.6), turned to -90 degrees
- moved R2 67.8 mm to (63.8, 35.9)
- moved C18 66.2 mm to (62.5, 35.6), turned to 90 degrees
- moved R1 65.6 mm to (63.9, 39.8)
- moved R6 58.8 mm to (73.9, 39.2), turned to 180 degrees
- moved R7 57.7 mm to (71.4, 48.5), turned to 180 degrees
- moved C21 54.8 mm to (74.6, 38.3)
- moved C22 54.3 mm to (71.4, 49.4), turned to 180 degrees
- moved J2 46.2 mm to (70.7, 41.2), turned to -90 degrees
- moved C23 45.9 mm to (87.4, 38.2)
- moved R8 45.8 mm to (87.4, 39.1)
- moved R9 45.4 mm to (84.8, 48.4), turned to 180 degrees
- moved C24 41.9 mm to (84.8, 49.5), turned to 180 degrees
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Connections:
- R1 pad 2: Net-(J2-Pad2) -> Net-(J2-Pad3)
- R2 pad 2: Net-(J2-Pad3) -> Net-(J2-Pad2)
Routing:
- net PA2: track 0.00 -> 41.7 mm, vias 0 -> 2
- net PA3: track 0.00 -> 32.9 mm, vias 0 -> 2
- net PA0: track 0.00 -> 22.0 mm, vias 0 -> 2
- net 3.3V: track 43.4 -> 64.7 mm, vias 0 -> 2
- net Net-(J3-Pad2): track 0.00 -> 20.8 mm
- net PA1: track 0.00 -> 19.3 mm, vias 0 -> 2
- net Net-(J3-Pad1): track 0.00 -> 19.3 mm
- net Net-(J3-Pad3): track 0.00 -> 11.1 mm
- net GND: track 0.00 -> 7.36 mm, vias 0 -> 3
- net Net-(J3-Pad4): track 0.00 -> 5.76 mm
- net Net-(J2-Pad2): track 0.00 -> 5.47 mm, vias 0 -> 1
- net Net-(J2-Pad3): track 0.00 -> 4.75 mm, vias 0 -> 1
- net 3.3VA: track 0.00 -> 4.28 mm
- net Net-(C21-Pad1): track 0.00 -> 4.08 mm
- net Net-(C23-Pad1): track 0.00 -> 4.00 mm
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- added copper zone on B.Cu, net GND
- added copper zone on F.Cu, net GND
Other:
- board outline added: 81.5 x 26.4 mm

Commit message: 15
Parts:
- moved Y1 0.98 mm to (46.8, 41.2)
- moved C19 0.80 mm to (50.7, 43.3)
- moved J1 0.77 mm to (27.2, 33.0)
- moved C20 0.23 mm to (51.5, 39.5)
Routing:
- net GND: track 7.36 -> 15.9 mm, vias 3 -> 17
- net 3.3VA: track 4.28 -> 8.60 mm
- net 3.3V: track 64.7 -> 62.6 mm
- net PD1: track 6.80 -> 8.19 mm
- net Net-(J1-VCC): track 4.83 -> 6.15 mm
- net PD0: track 6.38 -> 7.26 mm
- net Net-(J2-Pad2): track 5.47 -> 5.99 mm
