File: Эрозия прошивная/Платы/Плата управления прошивной эрозией/Плата управления прошивной эрозией.kicad_sch (KiCad schematic)
At the start: 37 parts, among them SW1 SW_Push, U3 STM32F103C8Tx, U8 HCPL-2630, U9 HCPL-2630, Y1 Crystal_GND24

Commit message: 1
Parts:
- removed C18, C21: 47pF, Capacitor_SMD:C_0603_1608Metric, symbol Device:C
- removed R6, R7: 100, Resistor_SMD:R_1206_3216Metric_Pad1.30x1.75mm_HandSolder, symbol Device:R
Connections:
- net SWCLK: now also J2.2
- net SWDIO: now also J2.3
Other:
- moved on the sheet: J2
